File: schematic/laundrysensor.sch (EAGLE design)
At the start: 15 parts, among them Q1 2N3904, Q2 2N3904

Commit message: working on i2s audio methods...
Parts:
- removed U$3: MCP4922-E/P, MCP4922-E_P:MCP4922-E/P
- added J1: Adafruit I2S amplifier MAX98357A, SparkFun-Connectors:CONN_07
- added R5: 100k, SparkFun-Resistors:100KOHM-HORIZ-1/4W-1%
Connections:
- removed net N$16: U$3.VOUTA
- removed net N$17: U$3.VOUTB
- net 3.3V: now also J1.6, R5.2; no longer U$3.AVSS, U$3.~LDAC
- net N$10: now also J1.1, WEMOS1.D4; no longer R4.1, WEMOS1.D3
- net N$2: now also R4.1, WEMOS1.D2; no longer U$3.SCK, WEMOS1.D5
- net N$4: now also WEMOS1.D3; no longer WEMOS1.D4
- net N$7: now also J1.4, R5.1; no longer U$3.SDI, WEMOS1.D7
- net N$8: now also J1.3, WEMOS1.RX; no longer U$3.~CS, WEMOS1.D8
- net N$9: now also J1.2, WEMOS1.D8; no longer U$3.~SHDN, WEMOS1.D2
- net VCC: now also J1.7; no longer U$3.VDD, U$3.VREFA, U$3.VREFB
Other:
- note added: "Free pins: A0, D5, D7"
- note added: "Vin GND SD Gain DIN BCLK LRC"
- note removed: "NOTE: D6 is MISO, which is unused by the 4922. It's unusable for other purposes here."
- note removed: "To amp (also /SHDN copied to amp)"
- moved on the sheet: R4

Commit message: wav playback working
Parts:
- removed U$4: NC_MARKER, NC_MARKER:NC_MARKER
Connections:
- net N$11: no longer U$4.P$1
Other:
- note added: "Free pins: A0, D5, D6, D7 - if we move D3 to A0, we could use a 23LC1024-ISN as external cache"
- note removed: "Free pins: A0, D5, D7"
Changed lines of the file:
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@@
 <part name="S1" library="bt_electromech" deviceset="SPST" device="_OFFBOARD_LG"/>
 <part name="GND3" library="SparkFun-PowerSymbols" deviceset="GND2" device=""/>
-<part name="U$4" library="NC_MARKER" deviceset="NC_MARKER" device=""/>
 <part name="U$5" library="NC_MARKER" deviceset="NC_MARKER" device=""/>
 <part name="D3" library="SparkFun-LED" deviceset="LED" device="3MM"/>
@@
 BCLK
 LRC</text>
-<text x="88.9" y="22.86" size="1.778" layer="91">Free pins: A0, D5, D7</text>
+<text x="88.9" y="22.86" size="1.778" layer="91">Free pins: A0, D5, D6, D7 - if we move D3 to A0, we could use a 23LC1024-ISN as external cache</text>
 </plain>
 <instances>
@@
 <attribute name="VALUE" x="93.98" y="104.902" size="1.778" layer="96" align="top-center"/>
 </instance>
-<instance part="U$4" gate="G$1" x="165.1" y="68.58" smashed="yes" rot="R90"/>
 <instance part="U$5" gate="G$1" x="172.72" y="68.58" smashed="yes" rot="R90"/>
 <instance part="D3" gate="G$1" x="139.7" y="134.62" smashed="yes" rot="R270">
@@
 <segment>
 <pinref part="WEMOS1" gate="D1" pin="D6"/>
-<pinref part="U$4" gate="G$1" pin="P$1"/>
 <wire x1="165.1" y1="73.66" x2="165.1" y2="71.12" width="0.1524" layer="91"/>
 </segment>

Commit message: schematic fixes
Parts:
- R1, R2: value 1k -> 100k
- R3, R4: value 1k -> 220
Connections:
- net N$5: now also D1.A; no longer D1.C
- net N$6: now also D2.A; no longer D2.C
- net VCC: now also D1.C, D2.C; no longer D1.A, D2.A
Other:
- moved on the sheet: D1, D2
Changed lines of the file:
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@@
 <part name="D1" library="opto-trans-siemens" library_urn="urn:adsk.eagle:library:317" deviceset="SFH205" device="" package3d_urn="urn:adsk.eagle:package:21801/1"/>
 <part name="D2" library="opto-trans-siemens" library_urn="urn:adsk.eagle:library:317" deviceset="SFH205" device="" package3d_urn="urn:adsk.eagle:package:21801/1"/>
-<part name="R1" library="SparkFun-Resistors" deviceset="1KOHM" device="-HORIZ-1/4W-5%" value="1k"/>
-<part name="R2" library="SparkFun-Resistors" deviceset="1KOHM" device="-HORIZ-1/4W-5%" value="1k"/>
+<part name="R1" library="SparkFun-Resistors" deviceset="1KOHM" device="-HORIZ-1/4W-5%" value="100k"/>
+<part name="R2" library="SparkFun-Resistors" deviceset="1KOHM" device="-HORIZ-1/4W-5%" value="100k"/>
 <part name="GND1" library="SparkFun-PowerSymbols" deviceset="GND2" device=""/>
 <part name="GND2" library="SparkFun-PowerSymbols" deviceset="GND2" device=""/>
@@
 <part name="D3" library="SparkFun-LED" deviceset="LED" device="3MM"/>
 <part name="D4" library="SparkFun-LED" deviceset="LED" device="3MM"/>
-<part name="R3" library="SparkFun-Resistors" deviceset="1KOHM" device="-HORIZ-1/4W-5%" value="1k"/>
-<part name="R4" library="SparkFun-Resistors" deviceset="1KOHM" device="-HORIZ-1/4W-5%" value="1k"/>
+<part name="R3" library="SparkFun-Resistors" deviceset="1KOHM" device="-HORIZ-1/4W-5%" value="220"/>
+<part name="R4" library="SparkFun-Resistors" deviceset="1KOHM" device="-HORIZ-1/4W-5%" value="220"/>
 <part name="J1" library="SparkFun-Connectors" deviceset="CONN_07" device="" value="Adafruit I2S amplifier MAX98357A"/>
 <part name="R5" library="SparkFun-Resistors" deviceset="100KOHM" device="-HORIZ-1/4W-1%" value="100k"/>
@@
 <attribute name="VALUE" x="43.72" y="76.66" size="1.778" layer="96"/>
 </instance>
-<instance part="D1" gate="1" x="50.8" y="116.84" smashed="yes">
-<attribute name="NAME" x="54.356" y="112.522" size="1.778" layer="95" rot="R90"/>
-<attribute name="VALUE" x="56.515" y="112.522" size="1.778" layer="96" rot="R90"/>
+<instance part="D1" gate="1" x="50.8" y="114.3" smashed="yes" rot="R180">
+<attribute name="NAME" x="47.244" y="118.618" size="1.778" layer="95" rot="R270"/>
+<attribute name="VALUE" x="45.085" y="118.618" size="1.778" layer="96" rot="R270"/>
 </instance>
-<instance part="D2" gate="1" x="33.02" y="86.36" smashed="yes">
-<attribute name="NAME" x="36.576" y="82.042" size="1.778" layer="95" rot="R90"/>
-<attribute name="VALUE" x="38.735" y="82.042" size="1.778" layer="96" rot="R90"/>
+<instance part="D2" gate="1" x="33.02" y="83.82" smashed="yes" rot="R180">
+<attribute name="NAME" x="29.464" y="88.138" size="1.778" layer="95" rot="R270"/>
+<attribute name="VALUE" x="27.305" y="88.138" size="1.778" layer="96" rot="R270"/>
 </instance>
 <instance part="R1" gate="G$1" x="63.5" y="119.38" smashed="yes" rot="R90">
@@
 <segment>
 <pinref part="Q1" gate="G$1" pin="B"/>
-<pinref part="D1" gate="1" pin="C"/>
 <wire x1="58.42" y1="104.14" x2="50.8" y2="104.14" width="0.1524" layer="91"/>
-<wire x1="50.8" y1="104.14" x2="50.8" y2="111.76" width="0.1524" layer="91"/>
+<pinref part="D1" gate="1" pin="A"/>
+<wire x1="50.8" y1="111.76" x2="50.8" y2="104.14" width="0.1524" layer="91"/>
 </segment>
 </net>
@@
 <segment>
 <pinref part="Q2" gate="G$1" pin="B"/>
-<pinref part="D2" gate="1" pin="C"/>
 <wire x1="38.1" y1="76.2" x2="33.02" y2="76.2" width="0.1524" layer="91"/>
-<wire x1="33.02" y1="76.2" x2="33.02" y2="81.28" width="0.1524" layer="91"/>
+<pinref part="D2" gate="1" pin="A"/>
+<wire x1="33.02" y1="81.28" x2="33.02" y2="76.2" width="0.1524" layer="91"/>
 </segment>
 </net>
@@
 <segment>
 <pinref part="R1" gate="G$1" pin="2"/>
-<pinref part="D1" gate="1" pin="A"/>
+<pinref part="U$1" gate="G$1" pin="VCC"/>
 <wire x1="63.5" y1="124.46" x2="50.8" y2="124.46" width="0.1524" layer="91"/>
-<wire x1="50.8" y1="124.46" x2="50.8" y2="119.38" width="0.1524" layer="91"/>
-<pinref part="U$1" gate="G$1" pin="VCC"/>
 <wire x1="50.8" y1="124.46" x2="25.4" y2="124.46" width="0.1524" layer="91"/>
-<junction x="50.8" y="124.46"/>
 <wire x1="25.4" y1="124.46" x2="25.4" y2="96.52" width="0.1524" layer="91"/>
 <junction x="25.4" y="124.46"/>
 <pinref part="R2" gate="G$1" pin="2"/>
-<pinref part="D2" gate="1" pin="A"/>
 <wire x1="43.18" y1="96.52" x2="33.02" y2="96.52" width="0.1524" layer="91"/>
-<wire x1="33.02" y1="96.52" x2="33.02" y2="88.9" width="0.1524" layer="91"/>
-<wire x1="25.4" y1="96.52" x2="33.02" y2="96.52" width="0.1524" layer="91"/>
+<pinref part="D2" gate="1" pin="C"/>
+<wire x1="33.02" y1="96.52" x2="25.4" y2="96.52" width="0.1524" layer="91"/>
+<wire x1="33.02" y1="88.9" x2="33.02" y2="96.52" width="0.1524" layer="91"/>
 <junction x="33.02" y="96.52"/>
+<pinref part="D1" gate="1" pin="C"/>
+<wire x1="50.8" y1="119.38" x2="50.8" y2="124.46" width="0.1524" layer="91"/>
+<junction x="50.8" y="124.46"/>
 </segment>
 <segment>

Commit message: abstract music player; wire up sensors and button for testing
Parts:
- Q1, Q2: value 2N3904 -> 2N4401
Connections:
- net N$4: now also WEMOS1.A0; no longer WEMOS1.D3
Other:
- note added: "Free pins: D3, D5, D6, D7 - we could use a 23LC1024-ISN as external cache on those"
- note removed: "Free pins: A0, D5, D6, D7 - if we move D3 to A0, we could use a 23LC1024-ISN as external cache"
Changed lines of the file:
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@@
 </classes>
 <parts>
-<part name="Q1" library="Transistor" library_urn="urn:adsk.eagle:library:16378713" deviceset="NPN" device="TO92-EBC" package3d_urn="urn:adsk.eagle:package:16378726/2" technology="_" value="2N3904"/>
-<part name="Q2" library="Transistor" library_urn="urn:adsk.eagle:library:16378713" deviceset="NPN" device="TO92-EBC" package3d_urn="urn:adsk.eagle:package:16378726/2" technology="_" value="2N3904"/>
+<part name="Q1" library="Transistor" library_urn="urn:adsk.eagle:library:16378713" deviceset="NPN" device="TO92-EBC" package3d_urn="urn:adsk.eagle:package:16378726/2" technology="_" value="2N4401"/>
+<part name="Q2" library="Transistor" library_urn="urn:adsk.eagle:library:16378713" deviceset="NPN" device="TO92-EBC" package3d_urn="urn:adsk.eagle:package:16378726/2" technology="_" value="2N4401"/>
 <part name="D1" library="opto-trans-siemens" library_urn="urn:adsk.eagle:library:317" deviceset="SFH205" device="" package3d_urn="urn:adsk.eagle:package:21801/1"/>
 <part name="D2" library="opto-trans-siemens" library_urn="urn:adsk.eagle:library:317" deviceset="SFH205" device="" package3d_urn="urn:adsk.eagle:package:21801/1"/>
@@
 BCLK
 LRC</text>
-<text x="88.9" y="22.86" size="1.778" layer="91">Free pins: A0, D5, D6, D7 - if we move D3 to A0, we could use a 23LC1024-ISN as external cache</text>
+<text x="88.9" y="22.86" size="1.778" layer="91">Free pins: D3, D5, D6, D7 - we could use a 23LC1024-ISN as external cache on those</text>
 </plain>
 <instances>
@@
 </segment>
 </net>
-<net name="N$4" class="0">
-<segment>
-<pinref part="WEMOS1" gate="D1" pin="D3"/>
-<wire x1="165.1" y1="104.14" x2="165.1" y2="114.3" width="0.1524" layer="91"/>
-<pinref part="S1" gate="G$1" pin="S"/>
-<wire x1="165.1" y1="114.3" x2="104.14" y2="114.3" width="0.1524" layer="91"/>
-</segment>
-</net>
 <net name="N$7" class="0">
 <segment>
@@
 </segment>
 </net>
+<net name="N$4" class="0">
+<segment>
+<pinref part="WEMOS1" gate="D1" pin="A0"/>
+<wire x1="157.48" y1="71.12" x2="157.48" y2="68.58" width="0.1524" layer="91"/>
+<wire x1="157.48" y1="68.58" x2="109.22" y2="68.58" width="0.1524" layer="91"/>
+<wire x1="109.22" y1="68.58" x2="109.22" y2="114.3" width="0.1524" layer="91"/>
+<pinref part="S1" gate="G$1" pin="S"/>
+<wire x1="109.22" y1="114.3" x2="104.14" y2="114.3" width="0.1524" layer="91"/>
+</segment>
+</net>

Commit message: updated schematic
Parts:
- removed U$5: NC_MARKER, NC_MARKER:NC_MARKER
- added R6: 10k, SparkFun-Resistors:10KOHM-HORIZ-1/4W-1%
Connections:
- removed net N$12: U$5.P$1, WEMOS1.3V3
- new net VCC_2: D1.C, D2.C, R1.2, R2.2, R6.2, WEMOS1.3V3
- net N$4: now also R6.1
- net VCC: no longer D1.C, D2.C, R1.2, R2.2
Changed lines of the file:
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@@
 <part name="GND1" library="SparkFun-PowerSymbols" deviceset="GND2" device=""/>
 <part name="GND2" library="SparkFun-PowerSymbols" deviceset="GND2" device=""/>
-<part name="U$1" library="bt" deviceset="VCC" device="" value="5v"/>
 <part name="WEMOS1" library="esp8266modules" deviceset="WEMOS-D1-MINI" device=""/>
 <part name="U$2" library="bt" deviceset="VCC" device="" value="5v"/>
 <part name="S1" library="bt_electromech" deviceset="SPST" device="_OFFBOARD_LG"/>
 <part name="GND3" library="SparkFun-PowerSymbols" deviceset="GND2" device=""/>
-<part name="U$5" library="NC_MARKER" deviceset="NC_MARKER" device=""/>
 <part name="D3" library="SparkFun-LED" deviceset="LED" device="3MM"/>
 <part name="D4" library="SparkFun-LED" deviceset="LED" device="3MM"/>
@@
 <part name="J1" library="SparkFun-Connectors" deviceset="CONN_07" device="" value="Adafruit I2S amplifier MAX98357A"/>
 <part name="R5" library="SparkFun-Resistors" deviceset="100KOHM" device="-HORIZ-1/4W-1%" value="100k"/>
+<part name="R6" library="SparkFun-Resistors" deviceset="10KOHM" device="-HORIZ-1/4W-1%" value="10k"/>
+<part name="SUPPLY1" library="SparkFun-PowerSymbols" deviceset="VCC_2" device=""/>
+<part name="SUPPLY2" library="SparkFun-PowerSymbols" deviceset="VCC_2" device=""/>
 </parts>
 <sheets>
@@
 <attribute name="VALUE" x="43.18" y="59.182" size="1.778" layer="96" align="top-center"/>
 </instance>
-<instance part="U$1" gate="G$1" x="25.4" y="124.46" smashed="yes">
-<attribute name="VALUE" x="25.4" y="132.588" size="1.778" layer="96" align="bottom-center"/>
-</instance>
 <instance part="WEMOS1" gate="D1" x="165.1" y="86.36" smashed="yes" rot="R90">
 <attribute name="NAME" x="152.4" y="76.2" size="1.778" layer="95" rot="R90"/>
@@
 <attribute name="VALUE" x="93.98" y="104.902" size="1.778" layer="96" align="top-center"/>
 </instance>
-<instance part="U$5" gate="G$1" x="172.72" y="68.58" smashed="yes" rot="R90"/>
 <instance part="D3" gate="G$1" x="139.7" y="134.62" smashed="yes" rot="R270">
 <attribute name="NAME" x="135.128" y="138.049" size="1.778" layer="95" font="vector"/>
@@
 <attribute name="NAME" x="149.86" y="49.784" size="1.778" layer="95" font="vector" align="bottom-center"/>
 <attribute name="VALUE" x="149.86" y="46.736" size="1.778" layer="96" font="vector" align="top-center"/>
+</instance>
+<instance part="R6" gate="G$1" x="157.48" y="60.96" smashed="yes">
+<attribute name="NAME" x="157.48" y="62.484" size="1.778" layer="95" font="vector" align="bottom-center"/>
+<attribute name="VALUE" x="157.48" y="59.436" size="1.778" layer="96" font="vector" align="top-center"/>
+</instance>
+<instance part="SUPPLY1" gate="G$1" x="25.4" y="129.54" smashed="yes">
+<attribute name="VALUE" x="25.4" y="132.334" size="1.778" layer="96" align="bottom-center"/>
+</instance>
+<instance part="SUPPLY2" gate="G$1" x="180.34" y="68.58" smashed="yes">
+<attribute name="VALUE" x="180.34" y="71.374" size="1.778" layer="96" align="bottom-center"/>
 </instance>
 </instances>
@@
 </net>
 <net name="VCC" class="0">
-<segment>
-<pinref part="R1" gate="G$1" pin="2"/>
-<pinref part="U$1" gate="G$1" pin="VCC"/>
-<wire x1="63.5" y1="124.46" x2="50.8" y2="124.46" width="0.1524" layer="91"/>
-<wire x1="50.8" y1="124.46" x2="25.4" y2="124.46" width="0.1524" layer="91"/>
-<wire x1="25.4" y1="124.46" x2="25.4" y2="96.52" width="0.1524" layer="91"/>
-<junction x="25.4" y="124.46"/>
-<pinref part="R2" gate="G$1" pin="2"/>
-<wire x1="43.18" y1="96.52" x2="33.02" y2="96.52" width="0.1524" layer="91"/>
-<pinref part="D2" gate="1" pin="C"/>
-<wire x1="33.02" y1="96.52" x2="25.4" y2="96.52" width="0.1524" layer="91"/>
-<wire x1="33.02" y1="88.9" x2="33.02" y2="96.52" width="0.1524" layer="91"/>
-<junction x="33.02" y="96.52"/>
-<pinref part="D1" gate="1" pin="C"/>
-<wire x1="50.8" y1="119.38" x2="50.8" y2="124.46" width="0.1524" layer="91"/>
-<junction x="50.8" y="124.46"/>
-</segment>
 <segment>
 <pinref part="U$2" gate="G$1" pin="VCC"/>
@@
 </segment>
 </net>
-<net name="N$12" class="0">
-<segment>
-<pinref part="WEMOS1" gate="D1" pin="3V3"/>
-<pinref part="U$5" gate="G$1" pin="P$1"/>
-<wire x1="172.72" y1="73.66" x2="172.72" y2="71.12" width="0.1524" layer="91"/>
-</segment>
-</net>
 <net name="N$13" class="0">
 <segment>
@@
 <pinref part="S1" gate="G$1" pin="S"/>
 <wire x1="109.22" y1="114.3" x2="104.14" y2="114.3" width="0.1524" layer="91"/>
-</segment>
-</net>
+<pinref part="R6" gate="G$1" pin="1"/>
+<wire x1="152.4" y1="60.96" x2="109.22" y2="60.96" width="0.1524" layer="91"/>
+<wire x1="109.22" y1="60.96" x2="109.22" y2="68.58" width="0.1524" layer="91"/>
+<junction x="109.22" y="68.58"/>
+</segment>
+</net>
+<net name="VCC_2" class="0">
+<segment>
+<pinref part="WEMOS1" gate="D1" pin="3V3"/>
+<wire x1="172.72" y1="73.66" x2="172.72" y2="71.12" width="0.1524" layer="91"/>
+<pinref part="R6" gate="G$1" pin="2"/>
+<wire x1="162.56" y1="60.96" x2="172.72" y2="60.96" width="0.1524" layer="91"/>
+<wire x1="172.72" y1="60.96" x2="172.72" y2="71.12" width="0.1524" layer="91"/>
+<junction x="172.72" y="71.12"/>
+<pinref part="SUPPLY2" gate="G$1" pin="VCC_2"/>
+<wire x1="172.72" y1="60.96" x2="180.34" y2="60.96" width="0.1524" layer="91"/>
+<wire x1="180.34" y1="60.96" x2="180.34" y2="68.58" width="0.1524" layer="91"/>
+<junction x="172.72" y="60.96"/>
+</segment>
+<segment>
+<pinref part="R1" gate="G$1" pin="2"/>
+<wire x1="63.5" y1="124.46" x2="50.8" y2="124.46" width="0.1524" layer="91"/>
+<wire x1="50.8" y1="124.46" x2="25.4" y2="124.46" width="0.1524" layer="91"/>
+<wire x1="25.4" y1="124.46" x2="25.4" y2="96.52" width="0.1524" layer="91"/>
+<pinref part="R2" gate="G$1" pin="2"/>
+<wire x1="43.18" y1="96.52" x2="33.02" y2="96.52" width="0.1524" layer="91"/>
+<pinref part="D2" gate="1" pin="C"/>
+<wire x1="33.02" y1="96.52" x2="25.4" y2="96.52" width="0.1524" layer="91"/>
+<wire x1="33.02" y1="88.9" x2="33.02" y2="96.52" width="0.1524" layer="91"/>
+<junction x="33.02" y="96.52"/>
+<pinref part="D1" gate="1" pin="C"/>
+<wire x1="50.8" y1="119.38" x2="50.8" y2="124.46" width="0.1524" layer="91"/>
+<junction x="50.8" y="124.46"/>
+<pinref part="SUPPLY1" gate="G$1" pin="VCC_2"/>
+<wire x1="25.4" y1="129.54" x2="25.4" y2="124.46" width="0.1524" layer="91"/>
+<junction x="25.4" y="124.46"/>
+</segment>
+</net>

Commit message: updated schematic after testing hardware...
Parts:
- removed Q1, Q2: 2N4401, Transistor:NPN_TO92-EBC
- removed R2: 100k, SparkFun-Resistors:1KOHM-HORIZ-1/4W-5%
- R1: value 100k -> 1k
Connections:
- removed net N$1: Q1.C, R1.1, WEMOS1.D1
- removed net N$6: D2.A, Q2.B
- new net N$12: D1.C, D2.C, R1.1
- net 3.3V: no longer Q1.E, Q2.E
- net N$3: now also D2.A; no longer Q2.C, R2.1
- net N$5: now also WEMOS1.D1; no longer Q1.B
- net VCC_2: no longer D1.C, D2.C, R2.2
Other:
- note added: "NOTE: Do not load down 3v3 output from the D1; its regulator is not sufficient for any load while operating WiFi"
- note removed: "NOTE: Do not use 3v3 output from the D1; its regulator is not sufficient for any load while operating WiFi"
- moved on the sheet: D1, D2, R1
